File: MCU-POWERSUPPLY.kicad_sch (KiCad schematic)
At the start: 10 parts, among them J3 Barrel_Jack, J4 USB_B_Micro, U4 LM2596S-5

Commit message: updates done
Parts:
- removed R2: R, symbol Device:R
- J4: footprint (none) -> Connector_USB:USB_Micro-B_Molex-105017-0001
Connections:
- net +5V: now also J4.4 (ID)
- net GND: no longer J4.5 (GND)
Other:
- moved on the sheet: J4
Changed lines of the file:
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@@
 	(wire
 		(pts
-			(xy 134.62 91.44) (xy 139.7 91.44)
+			(xy 134.62 91.44) (xy 152.4 91.44)
 		)
 		(stroke
@@
 		(pts
 			(xy 104.14 107.95) (xy 110.49 107.95)
-		)
-		(stroke
-			(width 0)
-			(type default)
-		)
-	)
-	(wire
-		(pts
-			(xy 147.32 91.44) (xy 152.4 91.44)
 		)
 		(stroke
@@
 	(symbol
 		(lib_id "Connector:USB_B_Micro")
-		(at 147.32 78.74 270)
+		(at 147.32 78.74 90)
+		(mirror x)
 		(unit 1)
 		(exclude_from_sim no)
@@
 		(dnp no)
 		(property "Reference" "J4"
-			(at 156.21 77.4699 90)
+			(at 138.43 77.4699 90)
 			(effects
 				(font
@@
 		)
 		(property "Value" "USB_B_Micro"
-			(at 157.226 78.74 0)
+			(at 137.414 78.74 0)
 			(effects
 				(font
@@
 			)
 		)
-		(property "Footprint" ""
-			(at 146.05 82.55 0)
+		(property "Footprint" "Connector_USB:USB_Micro-B_Molex-105017-0001"
+			(at 148.59 82.55 0)
 			(effects
 				(font
@@
 		)
 		(property "Datasheet" "~"
-			(at 146.05 82.55 0)
+			(at 148.59 82.55 0)
 			(effects
 				(font
@@
 		)
 		(property "Description" "USB Micro Type B connector"
+			(at 147.32 78.74 0)
+			(effects
+				(font
+					(size 1.27 1.27)
+				)
+				(hide yes)
+			)
+		)
+		(property "Sim.Library" "C:\\Users\\Victus\\Downloads\\165096554-36-1734035-2\\1734035-2_3D.dwg"
 			(at 147.32 78.74 0)
 			(effects
@@
 					(unit 1)
 				)
-			)
-		)
-	)
-	(symbol
-		(lib_id "Device:R")
-		(at 143.51 91.44 270)
-		(unit 1)
-		(exclude_from_sim no)
-		(in_bom yes)
-		(on_board yes)
-		(dnp no)
-		(property "Reference" "R2"
-			(at 143.51 93.726 90)
-			(effects
-				(font
-					(size 1.27 1.27)
-				)
-			)
-		)
-		(property "Value" "R"
-			(at 143.51 89.408 90)
-			(effects
-				(font
-					(size 1.27 1.27)
-				)
-			)
-		)
-		(property "Footprint" ""
-			(at 143.51 89.662 90)
-			(effects
-				(font
-					(size 1.27 1.27)
-				)
-				(hide yes)
-			)
-		)
-		(property "Datasheet" "~"
-			(at 143.51 91.44 0)
-			(effects
-				(font
-					(size 1.27 1.27)
-				)
-				(hide yes)
-			)
-		)
-		(property "Description" "Resistor"
-			(at 143.51 91.44 0)
-			(effects
-				(font
-					(size 1.27 1.27)
-				)
-				(hide yes)
-			)
-		)
-		(pin "1"
-		)
-		(pin "2"
-		)
-		(instances
-			(project "MCU-POWERSUPPLY"
-				(path "/f980154e-574c-4824-a575-d6afb7ffe96b"
-					(reference "R2")
-					(unit 1)
-				)

Commit message: added final schematics
Parts:
- F2: footprint (none) -> Fuse:Fuse_0402_1005Metric
Connections:
- net GND: now also J4.5 (GND)
Other:
- moved on the sheet: D2, F2, J3
Changed lines of the file:
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@@
 	)
 	(no_connect
-		(at 137.16 76.2)
-	)
-	(no_connect
-		(at 144.78 86.36)
+		(at 157.48 76.2)
 	)
 	(no_connect
 		(at 142.24 86.36)
 	)
+	(no_connect
+		(at 149.86 86.36)
+	)
 	(wire
 		(pts
@@
 	(wire
 		(pts
-			(xy 120.015 84.455) (xy 118.745 84.455)
+			(xy 120.65 83.82) (xy 118.11 83.82)
 		)
 		(stroke
@@
 	(wire
 		(pts
-			(xy 120.015 89.535) (xy 118.745 89.535)
-		)
-		(stroke
-			(width 0)
-			(type default)
-		)
-	)
-	(wire
-		(pts
 			(xy 149.86 113.03) (xy 153.67 113.03)
 		)
@@
 	(wire
 		(pts
+			(xy 120.65 88.9) (xy 118.11 88.9)
+		)
+		(stroke
+			(width 0)
+			(type default)
+		)
+	)
+	(wire
+		(pts
 			(xy 114.3 113.03) (xy 114.3 120.65)
 		)
@@
 	)
 	(label "+12V"
-		(at 120.015 84.455 0)
+		(at 120.65 83.82 0)
 		(effects
 			(font
@@
 	)
 	(label "GND"
-		(at 120.015 89.535 0)
+		(at 120.65 88.9 0)
 		(effects
 			(font
@@
 		(dnp no)
 		(property "Reference" "J4"
-			(at 138.43 77.4699 90)
+			(at 138.684 77.47 90)
 			(effects
 				(font
@@
 		)
 		(property "Value" "USB_B_Micro"
-			(at 137.414 78.74 0)
+			(at 131.318 78.486 0)
 			(effects
 				(font
@@
 	(symbol
 		(lib_id "Connector:Barrel_Jack")
-		(at 103.505 86.995 0)
+		(at 102.87 86.36 0)
 		(unit 1)
 		(exclude_from_sim no)
@@
 		(fields_autoplaced yes)
 		(property "Reference" "J3"
-			(at 103.505 78.105 0)
+			(at 102.87 77.47 0)
 			(effects
 				(font
@@
 		)
 		(property "Value" "Barrel_Jack"
-			(at 103.505 80.645 0)
+			(at 102.87 80.01 0)
 			(effects
 				(font
@@
 		)
 		(property "Footprint" ""
-			(at 104.775 88.011 0)
+			(at 104.14 87.376 0)
 			(effects
 				(font
@@
 		)
 		(property "Datasheet" "~"
-			(at 104.775 88.011 0)
+			(at 104.14 87.376 0)
 			(effects
 				(font
@@
 		)
 		(property "Description" "DC Barrel Jack"
-			(at 103.505 86.995 0)
+			(at 102.87 86.36 0)
 			(effects
 				(font
@@
 	(symbol
 		(lib_id "Device:D_Schottky")
-		(at 114.935 89.535 0)
+		(at 114.3 88.9 0)
 		(unit 1)
 		(exclude_from_sim no)
@@
 		(dnp no)
 		(property "Reference" "D2"
-			(at 115.443 92.837 0)
+			(at 114.808 92.202 0)
 			(effects
 				(font
@@
 		)
 		(property "Value" "D_Schottky"
-			(at 115.189 92.075 0)
+			(at 114.554 91.44 0)
 			(effects
 				(font
@@
 		)
 		(property "Footprint" ""
-			(at 114.935 89.535 0)
+			(at 114.3 88.9 0)
 			(effects
 				(font
@@
 		)
 		(property "Datasheet" "~"
-			(at 114.935 89.535 0)
+			(at 114.3 88.9 0)
 			(effects
 				(font
@@
 		)
 		(property "Description" "Schottky diode"
-			(at 114.935 89.535 0)
+			(at 114.3 88.9 0)
 			(effects
 				(font
@@
 	(symbol
 		(lib_id "Device:Fuse")
-		(at 114.935 84.455 270)
+		(at 114.3 83.82 270)
 		(unit 1)
 		(exclude_from_sim no)
@@
 		(dnp no)
 		(property "Reference" "F2"
-			(at 114.681 82.677 90)
+			(at 114.046 82.042 90)
 			(effects
 				(font
@@
 		)
 		(property "Value" "Fuse"
-			(at 113.665 82.169 90)
-			(effects
-				(font
-					(size 1.27 1.27)
-				)
-				(hide yes)
-			)
-		)
-		(property "Footprint" ""
-			(at 114.935 82.677 90)
+			(at 113.03 81.534 90)
+			(effects
+				(font
+					(size 1.27 1.27)
+				)
+				(hide yes)
+			)
+		)
+		(property "Footprint" "Fuse:Fuse_0402_1005Metric"
+			(at 114.3 82.042 90)
 			(effects
 				(font
@@
 		)
 		(property "Datasheet" "~"
-			(at 114.935 84.455 0)
+			(at 114.3 83.82 0)
 			(effects
 				(font
@@
 		)
 		(property "Description" "Fuse"
-			(at 114.935 84.455 0)
+			(at 114.3 83.82 0)
 			(effects
 				(font
@@
 	(symbol
 		(lib_id "power:GND")
-		(at 137.16 78.74 270)
+		(at 157.48 78.74 90)
 		(unit 1)
 		(exclude_from_sim no)
@@
 		(dnp no)
 		(property "Reference" "#PWR011"
-			(at 130.81 78.74 0)
+			(at 163.83 78.74 0)
 			(effects
 				(font
@@
 		)
 		(property "Value" "GND"
-			(at 137.668 81.026 90)
+			(at 157.226 74.422 90)
 			(effects
 				(font
@@
 		)
 		(property "Footprint" ""
-			(at 137.16 78.74 0)
+			(at 157.48 78.74 0)
 			(effects
 				(font
@@
 		)
 		(property "Datasheet" ""
-			(at 137.16 78.74 0)
+			(at 157.48 78.74 0)
 			(effects
 				(font
@@
 		)
 		(property "Description" "Power symbol creates a global label with name \"GND\" , ground"
-			(at 137.16 78.74 0)
-			(effects
-				(font
+			(at 157.48 78.74 0)
+			(effects
+				(font

Commit message: a
Parts:
- J3: footprint (none) -> Connector_BarrelJack:BarrelJack_Kycon_KLDX-0202-xC_Horizontal
Changed lines of the file:
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@@
 			)
 		)
-		(property "Footprint" ""
+		(property "Footprint" "Connector_BarrelJack:BarrelJack_Kycon_KLDX-0202-xC_Horizontal"
 			(at 104.14 87.376 0)
 			(effects

Commit message: a
Parts:
- C1: renamed from Cin2; footprint (none) -> Capacitor_THT:C_Disc_D3.0mm_W1.6mm_P2.50mm
- C2: renamed from COUT3; footprint (none) -> Capacitor_THT:C_Disc_D3.0mm_W1.6mm_P2.50mm
- D2: footprint (none) -> Diode_THT:D_DO-15_P12.70mm_Horizontal
- F2: footprint Fuse:Fuse_0402_1005Metric -> Fuse:Fuse_Bourns_MF-SM_7.98x5.44mm
- IN5826: footprint (none) -> Diode_THT:D_5W_P12.70mm_Horizontal
- J3: footprint Connector_BarrelJack:BarrelJack_Kycon_KLDX-0202-xC_Horizontal -> Connector_BarrelJack:BarrelJack_Wuerth_6941xx301002
- L3: footprint (none) -> Inductor_THT:L_Axial_L16.0mm_D6.3mm_P25.40mm_Horizontal_Fastron_VHBCC
Connections:
- net +5V: now also J4.1 (VBUS); no longer J4.4 (ID)
Changed lines of the file:
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@@
-	)
-	(junction
-		(at 158.75 113.03)
-		(diameter 0)
-		(color 0 0 0 0)
 	)
 	(junction
@@
 	)
 	(no_connect
-		(at 142.24 86.36)
+		(at 149.86 86.36)
 	)
 	(no_connect
-		(at 149.86 86.36)
+		(at 152.4 86.36)
 	)
 	(wire
@@
 	(wire
 		(pts
-			(xy 153.67 113.03) (xy 158.75 113.03)
-		)
-		(stroke
-			(width 0)
-			(type default)
-		)
-	)
-	(wire
-		(pts
-			(xy 134.62 91.44) (xy 152.4 91.44)
+			(xy 153.67 113.03) (xy 161.29 113.03)
 		)
 		(stroke
@@
 	(wire
 		(pts
+			(xy 158.75 87.63) (xy 142.24 87.63)
+		)
+		(stroke
+			(width 0)
+			(type default)
+		)
+	)
+	(wire
+		(pts
 			(xy 101.6 111.76) (xy 102.87 111.76)
 		)
@@
 	(wire
 		(pts
-			(xy 161.29 113.03) (xy 158.75 113.03)
+			(xy 142.24 87.63) (xy 142.24 86.36)
 		)
 		(stroke
@@
 	(wire
 		(pts
-			(xy 158.75 107.95) (xy 158.75 113.03)
-		)
-		(stroke
-			(width 0)
-			(type default)
-		)
-	)
-	(wire
-		(pts
 			(xy 104.14 120.65) (xy 110.49 120.65)
 		)
@@
 		(pts
 			(xy 110.49 120.65) (xy 114.3 120.65)
-		)
-		(stroke
-			(width 0)
-			(type default)
-		)
-	)
-	(wire
-		(pts
-			(xy 152.4 86.36) (xy 152.4 91.44)
 		)
 		(stroke
@@
 	)
 	(label "+5V"
-		(at 134.62 91.44 0)
+		(at 158.75 87.63 0)
 		(effects
 			(font
@@
 		(on_board yes)
 		(dnp no)
-		(property "Reference" "COUT3"
+		(property "Reference" "C2"
 			(at 154.178 114.808 0)
 			(effects
@@
 			)
 		)
-		(property "Footprint" ""
+		(property "Footprint" "Capacitor_THT:C_Disc_D3.0mm_W1.6mm_P2.50mm"
 			(at 154.6352 120.65 0)
 			(effects
@@
 			(project "MCU-POWERSUPPLY"
 				(path "/f980154e-574c-4824-a575-d6afb7ffe96b"
-					(reference "COUT3")
+					(reference "C2")
 					(unit 1)
 				)
@@
 	)
 	(symbol
-		(lib_id "power:PWR_FLAG")
-		(at 158.75 107.95 0)
-		(unit 1)
-		(exclude_from_sim no)
-		(in_bom yes)
-		(on_board yes)
-		(dnp no)
-		(property "Reference" "#FLG07"
-			(at 158.75 106.045 0)
-			(effects
-				(font
-					(size 1.27 1.27)
-				)
-				(hide yes)
-			)
-		)
-		(property "Value" "PWR_FLAG"
-			(at 158.75 104.14 0)
-			(effects
-				(font
-					(size 1.27 1.27)
-				)
-			)
-		)
-		(property "Footprint" ""
-			(at 158.75 107.95 0)
-			(effects
-				(font
-					(size 1.27 1.27)
-				)
-				(hide yes)
-			)
-		)
-		(property "Datasheet" "~"
-			(at 158.75 107.95 0)
-			(effects
-				(font
-					(size 1.27 1.27)
-				)
-				(hide yes)
-			)
-		)
-		(property "Description" "Special symbol for telling ERC where power comes from"
-			(at 158.75 107.95 0)
-			(effects
-				(font
-					(size 1.27 1.27)
-				)
-				(hide yes)
-			)
-		)
-		(pin "1"
-		)
-		(instances
-			(project "MCU-POWERSUPPLY"
-				(path "/f980154e-574c-4824-a575-d6afb7ffe96b"
-					(reference "#FLG07")
-					(unit 1)
-				)
-			)
-		)
-	)
-	(symbol
 		(lib_id "power:GND")
 		(at 127 121.92 0)
@@
 			)
 		)
-		(property "Footprint" "Connector_BarrelJack:BarrelJack_Kycon_KLDX-0202-xC_Horizontal"
+		(property "Footprint" "Connector_BarrelJack:BarrelJack_Wuerth_6941xx301002"
 			(at 104.14 87.376 0)
 			(effects
@@
 			)
 		)
-		(property "Footprint" ""
+		(property "Footprint" "Diode_THT:D_DO-15_P12.70mm_Horizontal"
 			(at 114.3 88.9 0)
 			(effects
@@
 		(on_board yes)
 		(dnp no)
-		(property "Reference" "Cin2"
+		(property "Reference" "C1"
 			(at 105.918 110.998 0)
 			(effects
@@
 			)
 		)
-		(property "Footprint" ""
+		(property "Footprint" "Capacitor_THT:C_Disc_D3.0mm_W1.6mm_P2.50mm"
 			(at 111.4552 116.84 0)
 			(effects
@@
 			(project "MCU-POWERSUPPLY"
 				(path "/f980154e-574c-4824-a575-d6afb7ffe96b"
-					(reference "Cin2")
+					(reference "C1")
 					(unit 1)
 				)
@@
 			)
 		)
-		(property "Footprint" ""
+		(property "Footprint" "Inductor_THT:L_Axial_L16.0mm_D6.3mm_P25.40mm_Horizontal_Fastron_VHBCC"
 			(at 146.05 113.03 0)
 			(effects
@@
 			)
 		)
-		(property "Footprint" "Fuse:Fuse_0402_1005Metric"
+		(property "Footprint" "Fuse:Fuse_Bourns_MF-SM_7.98x5.44mm"
 			(at 114.3 82.042 90)
 			(effects
@@
 		)
 		(property "Value" "GND"
-			(at 157.226 74.422 90)
+			(at 157.48 81.28 90)
 			(effects
 				(font
@@
 			)
 		)
-		(property "Footprint" ""
+		(property "Footprint" "Diode_THT:D_5W_P12.70mm_Horizontal"
 			(at 140.97 116.84 0)
 			(effects
